File: PCB/Prototype/densha_pico.kicad_pcb (KiCad board)
At the start: 2 copper layers, 100 x 100 mm, 23 parts, among them J1 NV3007, J2 Conn_01x04, J3 Conn_01x02, Q1 AO3400A, U1 PiPico_No_SWD, U2 CH221K, U3 DC/DC, U4 TMC2209, U5 8002A_Tap, U6 AS5600

Commit message: PCB v0.2
Parts:
- added C1: 0.1uF, Capacitor_SMD:C_0603_1608Metric_Pad1.08x0.95mm_HandSolder, F.Cu at (104.9, 150.9)
- added C2: 0.1uF, Capacitor_SMD:C_0603_1608Metric_Pad1.08x0.95mm_HandSolder, F.Cu at (127.1, 73.6)
- added C3: 0.1uF, Capacitor_SMD:C_0603_1608Metric_Pad1.08x0.95mm_HandSolder, F.Cu at (132.1, 129.7)
- added D3: SS34, Diode_SMD:D_SMA, F.Cu at (110.3, 152.9)
- added J4: NV3007_Stub, densha_pico:NV3007_Stub, F.Cu at (159.8, 106.4)
- added J5: Spin, densha_pico:SH1.0_4P_Solder_Combo, F.Cu at (132.3, 88.9)
- added J6: Spin, densha_pico:SH1.0_4P_Solder_Combo, F.Cu at (132.3, 80.4)
- added JP2: DIR, densha_pico:SmallJumper, F.Cu at (128.6, 133.4)
- added JP3: DIR, densha_pico:SmallJumper, F.Cu at (126.0, 133.4)
- added JP4: DIR, densha_pico:SmallJumper, F.Cu at (123.5, 133.4)
- J1: moved to F.Cu
- JP1: footprint Jumper:SolderJumper-2_P1.3mm_Open_RoundedPad1.0x1.5mm -> densha_pico:SmallJumper
- R5: value 5K1 -> 1K
- R6: value 5K1 -> 200K
- R8: value 3R3 -> 1K
- USB1: value HRO-TYPE-C-31-M-12 -> Data
- USB2: value HRO-TYPE-C-31-M-12 -> PD
- moved J1 32.6 mm to (136.3, 127.9), turned to 90 degrees
- moved R5 21.6 mm to (108.2, 148.3)
- moved J3 14.8 mm to (114.3, 75.6)
- moved R1 13.8 mm to (99.3, 84.2), turned to 0 degrees
- moved R4 13.2 mm to (100.8, 144.1), turned to 180 degrees
- moved R3 13.0 mm to (100.8, 142.5), turned to 180 degrees
- moved JP1 12.4 mm to (132.3, 69.4), turned to 180 degrees
- moved USB2 11.5 mm to (86.3, 144.4)
- moved R2 10.6 mm to (99.3, 86.5), turned to 0 degrees
- moved R7 9.40 mm to (129.3, 128.0)
- moved Q1 8.64 mm to (125.2, 128.0)
- moved U2 8.63 mm to (102.3, 147.4)
- moved R6 8.50 mm to (99.8, 150.9), turned to 0 degrees
- moved U6 6.73 mm to (132.3, 73.4), turned to 0 degrees
- moved J2 5.77 mm to (128.3, 156.4)
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Connections:
- J1 pad MP: (no net) -> GND
- R5 pad 2: VMOT -> Net-(D3-A)
- R6 pad 1: GND -> Net-(U2-CFG)
- R6 pad 2: Net-(U2-CFG) -> Net-(U2-VDD)
- U4 pad 4: unconnected-(U4-SPREAD-Pad4) -> Net-(JP2-A)
- U4 pad 5: /M_RX -> Net-(JP3-A)
- U4 pad 6: /M_RX -> Net-(JP4-A)
- USB2 pad 11: VMOT -> Net-(D3-A)
- USB2 pad 2: VMOT -> Net-(D3-A)
Routing:
- net +3V3: track 0.00 -> 161.6 mm, vias 0 -> 4
- net VBUS: track 0.00 -> 98.1 mm, vias 0 -> 2
- net /SCL: track 0.00 -> 63.8 mm, vias 0 -> 2
- net /AUDIO: track 0.00 -> 60.8 mm, vias 0 -> 1
- net /SDA: track 0.00 -> 59.0 mm, vias 0 -> 2
- net GND: track 0.00 -> 46.4 mm, vias 0 -> 20
- net /LCD_RST: track 0.00 -> 45.6 mm, vias 0 -> 2
- net VMOT: track 0.00 -> 40.3 mm
- net /LCD_SCL: track 0.00 -> 40.1 mm, vias 0 -> 2
- net /M_EN: track 0.00 -> 39.1 mm, vias 0 -> 1
- net /LCD_CS: track 0.00 -> 38.2 mm, vias 0 -> 2
- net /LCD_DC: track 0.00 -> 38.1 mm, vias 0 -> 2
- net /LCD_SDA: track 0.00 -> 37.3 mm, vias 0 -> 2
- net /LCD_LEDK: track 0.00 -> 37.2 mm, vias 0 -> 2
- net Net-(U1-USB2): track 0.00 -> 32.9 mm
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- added copper zone on B.Cu, net GND
- added copper zone on F.Cu, net GND
Other:
- board size 100 x 100 mm -> 90 x 100 mm
- board text added: "2B 2A 1A 1B"
- board text added: "5V to 6V+"
- board text added: "Densha Pico v0.2"
- board text added: "github.com/whowechina"

Commit message: PCB v0.3
Parts:
- added C4: 0.1uF, Capacitor_SMD:C_0603_1608Metric_Pad1.08x0.95mm_HandSolder, F.Cu at (131.2, 143.5)
- added R10: 1K, Resistor_SMD:R_0603_1608Metric_Pad0.98x0.95mm_HandSolder, F.Cu at (116.1, 131.1)
- added R11: 5.1K, Resistor_SMD:R_0603_1608Metric_Pad0.98x0.95mm_HandSolder, F.Cu at (116.1, 129.3)
- added R12: 1K, Resistor_SMD:R_0603_1608Metric_Pad0.98x0.95mm_HandSolder, F.Cu at (90.2, 131.2)
- added R13: 5.1K, Resistor_SMD:R_0603_1608Metric_Pad0.98x0.95mm_HandSolder, F.Cu at (90.2, 129.6)
- added R9: 0.1R, Inductor_SMD:L_1206_3216Metric_Pad1.42x1.75mm_HandSolder, F.Cu at (125.5, 146.7)
- added U7: INA219AxDCN, densha_pico:SOT-23-8_Thin, F.Cu at (127.3, 142.4)
- added Z1: 3.3V, Diode_SMD:D_SOD-123F, F.Cu at (107.8, 91.4)
- added Z2: 3.3V, Diode_SMD:D_SOD-123F, F.Cu at (112.9, 91.4)
Connections:
- U1 pad 32: unconnected-(U1-GPIO27_ADC1-Pad32) -> /Vsen1
- U1 pad 34: unconnected-(U1-GPIO28_ADC2-Pad34) -> /Vsen2
- U4 pad 16: VMOT -> Net-(U4-+VMOT)
Routing:
- net /Vsen1: track 0.00 -> 76.0 mm, vias 0 -> 2
- net /Vsen2: track 0.00 -> 51.2 mm, vias 0 -> 2
- net /SDA: track 59.0 -> 99.9 mm, vias 2 -> 4
- net /SCL: track 63.8 -> 104.3 mm, vias 2 -> 4
- net +3V3: track 161.6 -> 177.9 mm, vias 4 -> 5
- net Net-(U4-+VMOT): track 0.00 -> 14.5 mm
- net Net-(D3-A): track 31.4 -> 45.0 mm, vias 2 -> 3
- net GND: track 46.4 -> 55.4 mm, vias 20 -> 24
- net /M_EN: track 39.1 -> 45.9 mm, vias 1 -> 0
- net VBUS: track 98.1 -> 103.0 mm
- net /M_DIR: track 24.1 -> 22.2 mm
- net VMOT: track 40.3 -> 41.0 mm
Other:
- board text added: "Densha Pico v0.3"
- board text removed: "Densha Pico v0.2"
