File: PCB/Prototype/densha_pico.kicad_sch (KiCad schematic)
At the start: 23 parts, among them J1 NV3007, J2 Conn_01x04, J3 Conn_01x02, Q1 AO3400A, U1 PiPico_No_SWD, U2 CH221K, U3 DC/DC, U4 TMC2209, U5 8002A_Tap, U6 AS5600

Commit message: PCB v0.2
Parts:
- added C1, C2, C3: 0.1uF, Capacitor_SMD:C_0603_1608Metric_Pad1.08x0.95mm_HandSolder, symbol Device:C
- added D3: SS34, Diode_SMD:D_SMA, symbol Diode:SS34
- added J4: NV3007_Stub, densha_pico:NV3007_Stub, symbol densha_pico:NV3007_Stub
- added J5, J6: Spin, densha_pico:SH1.0_4P_Solder_Combo, symbol Connector_Generic:Conn_01x04
- added JP2, JP3, JP4: DIR, densha_pico:SmallJumper, symbol Jumper:SolderJumper_2_Open
- J3: footprint Solder_2P -> densha_pico:Solder_2P
- JP1: footprint Jumper:SolderJumper-2_P1.3mm_Open_RoundedPad1.0x1.5mm -> densha_pico:SmallJumper
- R5: value 5K1 -> 1K
- R6: value 5K1 -> 200K
- R8: value 3R3 -> 1K
- USB1: value HRO-TYPE-C-31-M-12 -> Data
- USB2: value HRO-TYPE-C-31-M-12 -> PD
Connections:
- net +3V3: now also C2.1, C3.1, J5.1 (Pin_1), J6.1 (Pin_1)
- net GND: now also J1.MP (Mouting), C1.2, C2.2, C3.2, J5.4 (Pin_4), J6.4 (Pin_4); no longer R6.1
- net M_RX: now also JP2.2 (B), JP3.2 (B), JP4.2 (B); no longer U4.5 (UART), U4.6 (UART)
- net SCL: now also J5.2 (Pin_2), J6.2 (Pin_2)
- net SDA: now also J5.3 (Pin_3), J6.3 (Pin_3)
- net VMOT: now also D3.1 (K); no longer R5.2, USB2.11 (VBUS), USB2.2 (VBUS)
- net at R5.1, U2.1 (VDD): now also R6.2, C1.1
- net at U2.6 (CFG): now also R6.1; no longer R6.2
- net at U4.4 (SPREAD): now also JP2.1 (A)
- new net: JP4.1 (A), U4.6 (UART)
- new net: D3.2 (A), R5.2, USB2.11 (VBUS), USB2.2 (VBUS)
- new net: JP3.1 (A), U4.5 (UART)
- no-connect marks 14 -> 13
Other:
- moved on the sheet: JP1, R5, R6, U2, U6

Commit message: PCB v0.3
Parts:
- added C4: 0.1uF, Capacitor_SMD:C_0603_1608Metric_Pad1.08x0.95mm_HandSolder, symbol Device:C
- added R10, R12: 1K, Resistor_SMD:R_0603_1608Metric_Pad0.98x0.95mm_HandSolder, symbol Device:R_Small
- added R11, R13: 5.1K, Resistor_SMD:R_0603_1608Metric_Pad0.98x0.95mm_HandSolder, symbol Device:R_Small
- added R9: 0.1R, Inductor_SMD:L_1206_3216Metric_Pad1.42x1.75mm_HandSolder, symbol Device:R_Small
- added U7: INA219AxDCN, densha_pico:SOT-23-8_Thin, symbol Sensor_Energy:INA219AxDCN
- added Z1, Z2: 3.3V, Diode_SMD:D_SOD-123F, symbol Device:D_Zener
Connections:
- net +3V3: now also C4.1, U7.4 (VS)
- net GND: now also C4.2, R11.2, R13.2, U7.3 (GND), U7.7 (A0), U7.8 (A1), Z1.2 (A), Z2.2 (A)
- net SCL: now also U7.5 (SCL)
- net SDA: now also U7.6 (SDA)
- net VMOT: now also R10.1, R9.2, U7.1 (IN+); no longer U4.16 (+VMOT)
- net at D3.2 (A), R5.2, USB2.11 (VBUS)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: now also R12.1
- net Vsen1: now reaches U1.32 (GPIO27_ADC1)
- net Vsen1: now also R10.2, R11.1, Z2.1 (K)
- net Vsen2: now reaches U1.34 (GPIO28_ADC2)
- net Vsen2: now also R12.2, R13.1, Z1.1 (K)
- new net: R9.1, U4.16 (+VMOT), U7.2 (IN-)
Other:
- moved on the sheet: C2, J2, J5, J6, JP1, JP2, JP3, JP4, U4, U6
